File: SHABlindRfShield.brd (EAGLE design)
At the start: 59.7 x 53.3 mm, 23 parts, among them J1 Digital_0_7, J2 Analog, J3 Digital_8_13, J4 Power

Commit message: Routing and silkscreen
Parts:
- removed ANT: M01PTH, freetronics:1X01
- removed LED3: RED, freetronics:LED-0603
- removed PADS_5V, PADS_GND: M16PTH, freetronics-2:1X16
- removed RX1: RXB1SIL, PracticalArduino:RX-B1
- added ANT1, ANT2: M01PTH, freetronics:1X01
- added C2: 10uF 0805, freetronics-jon:C0805
- added IC3: RXB1, freetronics-master-v1:RX-B1-SHORT-FLAT
- added IC4: TX-C1FLAT, freetronics-jon:TX-C1-FLAT
- C1: value 100nF -> 100nF 0603
- R4: value 820R -> 1K
- S1: device freetronics-master-v1:TACTILE_SWITCH_SMD_2PIN_TINY -> freetronics-jon:TACTILE_SWITCH_SMD_2PIN_TINY
- moved LED1 47.1 mm to (3.21, 4.95)
- moved LED2 41.1 mm to (46.1, 42.4)
- moved U$4 40.0 mm to (38.5, 16.1), turned to 270 degrees
- moved U$5 36.5 mm to (20.5, 41.0), turned to 270 degrees
- moved R3 36.2 mm to (42.4, 42.4), turned to 180 degrees
- moved R4 29.9 mm to (38.9, 41.7), turned to 270 degrees
- moved C1 29.7 mm to (27.4, 11.4), turned to 0 degrees
- moved R1 13.0 mm to (3.30, 7.62), turned to 0 degrees
- moved R2 10.9 mm to (24.1, 25.4), turned to 180 degrees
- moved J4 7.62 mm to (11.4, 2.54)
- moved SL4 7.62 mm to (11.4, 7.62)
- moved S1 7.62 mm to (7.62, 5.08)
- moved J1 7.62 mm to (47.0, 50.8)
- moved J2 7.62 mm to (34.3, 2.54)
- moved J3 7.62 mm to (25.1, 50.8)
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Connections:
- new net N$4: ANT2.1, IC4.1
- net 5V: now also C2.2, IC3.4, IC4.2; no longer PADS_5V.1, PADS_5V.10, PADS_5V.11, PADS_5V.12, PADS_5V.13, PADS_5V.14, PADS_5V.15, PADS_5V.16, PADS_5V.2, PADS_5V.3, PADS_5V.4, PADS_5V.5, PADS_5V.6, PADS_5V.7, PADS_5V.8, PADS_5V.9, RX1.12, RX1.22
- net D5: now also R4.1
- net D7: no longer R4.2
- net GND: now also C2.1, IC3.1, IC3.5, IC4.4; no longer LED3.C, PADS_GND.1, PADS_GND.10, PADS_GND.11, PADS_GND.12, PADS_GND.13, PADS_GND.14, PADS_GND.15, PADS_GND.16, PADS_GND.2, PADS_GND.3, PADS_GND.4, PADS_GND.5, PADS_GND.6, PADS_GND.7, PADS_GND.8, PADS_GND.9, RX1.10, RX1.11, RX1.25
- net N$135: now also IC3.3; no longer RX1.23
- net N$3: now also ANT1.1, IC3.6; no longer LED3.A, R4.1
- net N$6: now also IC4.3, R4.2; no longer ANT.1, RX1.9
Routing:
- net N$1: track 49.6 -> 2.70 mm
- net 5V: track 109.1 -> 63.9 mm
- net D7: track 46.8 -> 5.08 mm, vias 1 -> 0
- net N$2: track 43.4 -> 2.19 mm
- net N$3: track 35.8 -> 8.67 mm
- net D8: track 47.0 -> 25.5 mm
- net N$135: track 29.3 -> 10.5 mm, vias 1 -> 0
- net D6: track 54.2 -> 41.1 mm, vias 1 -> 0
- net D5: track 5.08 -> 12.1 mm
- net N$4: track 0.00 -> 5.08 mm, vias 1 -> 0
- net N$6: track 8.15 -> 5.50 mm
Other:
- board size 59.7 x 53.3 mm -> 49.5 x 53.3 mm
- board text added: "(C)2015 SuperHouse Automation P/L"
- board text added: "433MHz RF Shield v1.0"
- board text added: "ACTIVITY"
- board text added: "D0: Serial RX D1: Serial TX D5: RF TX D6: Activity LED D8: RF RX"
- board text added: "RX"
- board text added: "SKU: RFSHIELD"
- board text added: "TX"
- board text added: "TXC1"
- board text added: "www.superhouse.tv/rfshield"
- board text removed: "(C)2012 Freetronics Pty Ltd"
- board text removed: "1"
- board text removed: "17"
- board text removed: "Licensed under the TAPR"
- board text removed: "Open Hardware License"
- board text removed: "Receiver Shield v4.0"
- board text removed: "SKU: SH-RECEIVER"
- board text removed: "freetronics"
- board text removed: "www.freetronics.com"
- board text removed: "www.freetronics.com/receiver"
- board text removed: "www.tapr.org/OHL"
