File: SHABlindRfShield.sch (EAGLE design)
At the start: 23 parts, among them J1 Digital_0_7, J2 Analog, J3 Digital_8_13, J4 Power

Commit message: Routing and silkscreen
Parts:
- removed LED3: RED, freetronics:LED0603
- removed PADS_5V, PADS_GND: M16PTH, freetronics-2:M16PTH
- removed RX1: RXB1SIL, PracticalArduino:RXB1SIL
- added ANT2: M01PTH, freetronics:M01PTH
- added C2: 10uF 0805, freetronics-jon:C-EUC0805
- added IC3: RXB1, freetronics-master-v1:RXB1SHORTFLAT
- added IC4: TX-C1FLAT, freetronics-jon:TX-C1FLAT
- C1: value 100nF -> 100nF 0603
- R4: value 820R -> 1K
- S1: device freetronics-master-v1:TAC_SWITCH_2PIN -> freetronics-jon:TAC_SWITCH_2PIN
- renumbered ANT to ANT1
Connections:
- new net N$4: ANT2.1, IC4.ANT
- net 5V: now also C2.2, IC3.VCC, IC4.VCC; no longer PADS_5V.1, PADS_5V.10, PADS_5V.11, PADS_5V.12, PADS_5V.13, PADS_5V.14, PADS_5V.15, PADS_5V.16, PADS_5V.2, PADS_5V.3, PADS_5V.4, PADS_5V.5, PADS_5V.6, PADS_5V.7, PADS_5V.8, PADS_5V.9, RX1.VCC, RX1.VCC2
- net D5: now also R4.1
- net D7: no longer R4.2
- net GND: now also C2.1, IC3.GND1, IC3.GND2, IC4.GND; no longer LED3.C, PADS_GND.1, PADS_GND.10, PADS_GND.11, PADS_GND.12, PADS_GND.13, PADS_GND.14, PADS_GND.15, PADS_GND.16, PADS_GND.2, PADS_GND.3, PADS_GND.4, PADS_GND.5, PADS_GND.6, PADS_GND.7, PADS_GND.8, PADS_GND.9, RX1.GND, RX1.GND2, RX1.GND3
- net N$135: now also IC3.DATA2; no longer RX1.DATA
- net N$3: now also ANT1.1, IC3.ANT; no longer LED3.A, R4.1
- net N$6: now also IC4.DATA, R4.2; no longer ANT1.1, RX1.ANT
Other:
- note added: "Blind RF Shield"
- note added: "D0: Serial RX D1: Serial TX D5: RF TX data D6: LED D8: RF RX data"
- note added: "SKU: RFSHIELD"
- note added: "V1.0 (2015-11-18)"
- note added: "www.superhouse.tv/rfshield"
- note removed: "Freetronics Receiver Shield"
- note removed: "SKU: SH-RECEIVER"
- note removed: "V4.0 (2012-12-06)"
- note removed: "www.freetronics.com/receiver-shield"
- moved on the sheet: C1, R4
